File: PCB/PCB_Gantry/F2.kicad_sch (KiCad schematic)
At the start: 67 parts, among them J1 Screw_Terminal_01x02, J2 esp32 30 pin, J3 JST, J4 JST, J5 JST, U10 DRV8825_STEPPER_MOTOR_DRIVER_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, U11 DRV8825_STEPPER_MOTOR_DRIVER_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, U12 DRV8825_STEPPER_MOTOR_DRIVER_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

Commit message: Updated Schematic with labels
Parts:
- added C39: 10 uF, symbol Device:C_Small
- added C40: 100 nF, symbol Device:C_Small
- added C41: 220 pF, symbol Device:C_Small
- added C42: NS, symbol Device:C_Small
- added C43: 22 uF, symbol Device:C_Small
- added C44: 100 uF, symbol Device:C
- added C45: 0.1 uF, symbol Device:C
- added D8: D_Zener_Small, symbol Device:D_Zener_Small
- added L8: L_Small, symbol Device:L_Small
- added M1: Motor_DC, symbol Motor:Motor_DC
- added R43: 24.9k, symbol Device:R
- added R44: 200k, symbol Device:R
- added R45: 100k, symbol Device:R
- added R46: 68.1k, symbol Device:R
- added R47: 10k, symbol Device:R
- added R48: 140k, symbol Device:R
- added R49: 0.1 k, symbol Device:R
- added SW1: SW_SPDT_XKB_DMx-xxxx-1, symbol Switch:SW_SPDT_XKB_DMx-xxxx-1
- added U13: ~, symbol Components:MP1584
Connections:
- net Earth: now also U10.15 (GND_MOT), U11.15 (GND_MOT), U12.15 (GND_MOT), C39.1, C42.2, C43.1, D8.2 (A), M1.2 (-), R43.2, R44.2, R46.2, R47.2, R49.2, U13. (COMP); no longer C16.2, C21.2, C26.2, C31.2, J1.2 (Pin_2), J2.14 (GND), R21.1, R27.1, R33.1, R39.1
- net 3v3: now reaches J2.16 (3V3), U10.2 (M0), U10.3 (M1), U10.4 (M2), U10.5 (~{RST}), U10.6 (~{SLP}), U11.2 (M0), U11.3 (M1), U11.4 (M2), U11.5 (~{RST}), U11.6 (~{SLP}), U12.2 (M0), U12.3 (M1), U12.4 (M2), U12.5 (~{RST}), U12.6 (~{SLP})
- net 3v3: now also SW1.1 (A)
- net D19: now reaches J2.25 (D19), U11.7 (STEP)
- net D18: now reaches J2.24 (D18), U11.8 (DIR)
- net GND_L: now reaches J2.17 (GND), U10.9 (GND), U11.9 (GND), U12.9 (GND)
- net D32: now reaches J2.6 (D32)
- net D32: now also U12.8 (DIR); no longer U12.7 (STEP)
- net D33: now reaches J2.7 (D33)
- net D33: now also U12.7 (STEP); no longer U12.8 (DIR)
- net D4: now reaches J2.20 (D4), U10.7 (STEP)
- net D2: now reaches J2.19 (D2), U10.8 (DIR)
- net at J2.9 (D26): now also SW1.2 (B), SW1.3 (C)
- new net: C43.2, C44.1, C44.2, C45.1, L8.2, M1.1 (+), R48.2
- new net: C41.2, R46.1
- new net: C40.2, D8.1 (K), L8.1, U13. (COMP)
- new net: R43.1, R45.2, U13. (COMP)
- new net: C41.1, C42.1, U13. (COMP)
- new net: C45.2, R49.1
- new net: R47.1, R48.1, U13. (COMP)
- new net: R44.1, U13. (COMP)
- new net 28V: C16.2, C21.2, C26.2, C31.2, C39.2, J1.2 (Pin_2), R21.1, R27.1, R33.1, R39.1, R45.1, U13. (COMP), U6. (COMP), U7. (COMP), U8. (COMP), U9. (COMP)
Other:
- note added: "Not for First Prototype"
